Commit message: use custom joint_trajectory_controller successfully

File: mycobot_description/urdf/mech/mycobot_280_arm.urdf.xacro (robot description, xacro)
@@ -1,5 +1,6 @@
 <?xml version="1.0"?>
 <robot xmlns:xacro="http://www.ros.org/wiki/xacro">
-  <xacro:property name="joint_effort" value="56.0"/>
+  <!-- <xacro:property name="joint_effort" value="56.0"/> -->
+  <xacro:property name="joint_effort" value="1000.0"/>
   <xacro:property name="joint_velocity" value="2.792527"/>
   <xacro:property name="joint_damping" value="0.0"/>
